Commit message: add end effector

File: install/tros_sldworks_pkg/share/tros_sldworks_pkg/urdf/robot_description.urdf (robot description, URDF)
Before this commit: robot tros_sldworks_pkg, 12 links, 11 joints
Links:
- added link arm_end_effector_spin_link, mass 0.33685; collision mesh filename=package://tros_sldworks_pkg/meshes/arm_end_effector_spin_li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; visual mesh filename=package://tros_sldworks_pkg/meshes/arm_end_effector_spin_li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
- added link arm_end_effector_turn_link, mass 0.0545581570050041; collision mesh filename=package://tros_sldworks_pkg/meshes/arm_end_effector_turn_li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; visual mesh filename=package://tros_sldworks_pkg/meshes/arm_end_effector_turn_li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
- link arm_base_turret_link: mass 1.54125416646532 -> 1.54125416810131
- link arm_mid_link: mass 0.98691392916891 -> 1.17448790322858
- link arm_turret_link: mass 2.22661607727245 -> 0
- link front_left_link: mass 12.2088239451308 -> 12.209
- link left_rotatable_link: mass 3.40229054558914 -> 3.40229054558915
Joints:
- added joint arm_end_effector_spin_joint: type continuous, parent arm_end_effector_turn_link, child arm_end_effector_spin_link, origin xyz=0.02119 0.011271 -0.0037291 rpy=1.5708 -1.2555 -1.0709, axis 0 0 -1
- added joint arm_end_effector_turn_joint: type revolute, parent arm_mid_link, child arm_end_effector_turn_link, origin xyz=0.5747 -0.062022 0.05667 rpy=2.8595 0.14022 0.34467, axis 0 0 -1, limit lower=-3.14 upper=3.14 effort=0 velocity=0
- joint arm_base_turret_joint: limit lower=-3.1419 upper=3.1419 effort=0 velocity=0 -> lower=-3.14 upper=3.14 effort=0 velocity=0; origin xyz=-0.0942026527316038 0.0718895770090404 0.0863499899999998 rpy=1.5707963267949 0 -2.2226525007642 -> xyz=-0.094203 0.07189 0.08635 rpy=1.5708 0 -2.2227
- joint arm_mid_joint: limit lower=-3.1419 upper=3.1419 effort=0 velocity=0 -> lower=-3.14 upper=3.14 effort=0 velocity=0; origin xyz=0 0.615200000000052 -0.0202624999999994 rpy=-3.14159265358979 0 0 -> xyz=0 0.6152 -0.020262 rpy=-3.1416 0 0
- joint arm_turret_joint: origin xyz=0 0.189388974321119 0 rpy=1.5707963267949 0 -3.14159265358979 -> xyz=0 0.19 0 rpy=1.5708 0 -3.1416
- joint chassis_joint: origin xyz=0.0 0.0 0.0 rpy=1.5708 0.0 0.0 -> xyz=0.0 0.0 0.0 rpy=1.5708 0 0
- joint front_left_joint: origin xyz=-0.399129309591516 -0.248184999999998 0.0846516733300001 rpy=-3.14159265358979 0 -3.14159265358979 -> xyz=-0.39913 -0.24818 0.084652 rpy=-3.1416 0 -3.1416
- joint left_rotatable_joint: limit lower=-1.57 upper=1.57 effort=0 velocity=1 -> lower=-1.57 upper=1.57 effort=0 velocity=0
- joint lidar_joint: axis 0 0 0 -> 0 1 0; type fixed -> continuous
- joint right_rotatable_joint: limit lower=-1.57 upper=1.57 effort=0 velocity=1 -> lower=-1.57 upper=1.57 effort=0 velocity=0
