Commit message: gazebo lidar sim

File: urdf/robot_description.urdf (robot description, URDF)
Before this commit: robot tros_sldworks_pkg, 14 links, 13 joints
Links:
- link arm_turret_link: mass 0 -> 1
Joints:
- joint lidar_joint: axis 0 1 0 -> (none); type continuous -> fixed

Commit message: joystick simulation

File: urdf/robot_description.urdf (robot description, URDF)
Before this commit: robot tros_sldworks_pkg, 14 links, 13 joints
Joints:
- joint front_right_joint: axis 0 0 -1 -> 0 0 1
- joint rear_right_joint: axis 0 0 -1 -> 0 0 1
