Commit message: ros2_control demo working

File: urdf/robot_description.urdf.xacro (robot description, xacro)
@@ -1,4 +1,4 @@
 <?xml version="1.0"?>
-<robot
+<robot xmlns:xacro="http://ros.org"
   name="tros_sldworks_pkg">
   <link name="base_link"></link>
@@ -773,22 +773,64 @@
       damping="0.4" />
   </joint>
+  <!-- <gazebo> -->
+    <!-- <plugin filename="gz-sim-diff-drive-system" name="gz::sim::systems::DiffDrive"> -->
+      <!-- <left_joint>front_left_joint</left_joint> -->
+      <!-- <left_joint>rear_left_joint</left_joint> -->
+      <!-- <right_joint>front_right_joint</right_joint> -->
+      <!-- <right_joint>rear_right_joint</right_joint> -->
+      <!-- <wheel_separation>0.4</wheel_separation> -->
+      <!-- <wheel_radius>0.15</wheel_radius> -->
+      <!-- <publish_odom>true</publish_odom> -->
+      <!-- <publish_odom_tf>true</publish_odom_tf> -->
+      <!-- <publish_wheel_tf>true</publish_wheel_tf> -->
+      <!-- <odom_publish_frequency>50</odom_publish_frequency> -->
+      <!-- <topic>/cmd_vel</topic> -->
+      <!-- <odom_topic>/odom</odom_topic> -->
+      <!-- <tf_topic>/tf</tf_topic> -->
+      <!-- <frame_id>odom</frame_id> -->
+      <!-- <child_frame_id>base_link</child_frame_id> -->
+    <!-- </plugin> -->
+  <!-- </gazebo> -->
   <gazebo>
-    <plugin filename="gz-sim-diff-drive-system" name="gz::sim::systems::DiffDrive">
-      <left_joint>front_left_joint</left_joint>
-      <left_joint>rear_left_joint</left_joint>
-      <right_joint>front_right_joint</right_joint>
-      <right_joint>rear_right_joint</right_joint>
-      <wheel_separation>0.4</wheel_separation>
-      <wheel_radius>0.15</wheel_radius>
-      <publish_odom>true</publish_odom>
-      <publish_odom_tf>true</publish_odom_tf>
-      <publish_wheel_tf>true</publish_wheel_tf>
-      <odom_publish_frequency>50</odom_publish_frequency>
-      <topic>/cmd_vel</topic>
-      <odom_topic>/odom</odom_topic>
-      <tf_topic>/tf</tf_topic>
-      <frame_id>odom</frame_id>
-      <child_frame_id>base_link</child_frame_id>
+    <plugin filename="libgz_ros2_control-system.so" name="gz_ros2_control::GazeboSimROS2ControlPlugin">
+      <parameters>$(find tros_sldworks_pkg)/config/test_controller.yaml</parameters>
     </plugin>
   </gazebo>
+  <ros2_control name="GZ System" type="system">
+    <hardware>
+      <plugin>gz_ros2_control/GazeboSimSystem</plugin>
+    </hardware>
+    <joint name="front_right_joint">
+      <command_interface name="velocity">
+        <param name="min">-10</param>
+        <param name="max">10</param>
+      </command_interface>
+      <state_interface name="velocity"></state_interface>
+      <state_interface name="position"></state_interface>
+    </joint>
+    <joint name="front_left_joint">
+      <command_interface name="velocity">
+        <param name="min">-10</param>
+        <param name="max">10</param>
+      </command_interface>
+      <state_interface name="velocity"></state_interface>
+      <state_interface name="position"></state_interface>
+    </joint>
+    <joint name="rear_right_joint">
+      <command_interface name="velocity">
+        <param name="min">-10</param>
+        <param name="max">10</param>
+      </command_interface>
+      <state_interface name="velocity"></state_interface>
+      <state_interface name="position"></state_interface>
+    </joint>
+    <joint name="rear_left_joint">
+      <command_interface name="velocity">
+        <param name="min">-10</param>
+        <param name="max">10</param>
+      </command_interface>
+      <state_interface name="velocity"></state_interface>
+      <state_interface name="position"></state_interface>
+    </joint>
+  </ros2_control>
 </robot>

Commit message: added arm joints, fixed lidar

File: urdf/robot_description.urdf.xacro (robot description, xacro)
@@ -449,6 +449,6 @@
             <samples>16</samples>
             <resolution>1</resolution>
-            <min_angle>-0.2617993877991494</min_angle> <!-- -15 degrees -->
-            <max_angle>0.2617993877991494</max_angle>  <!-- +15 degrees -->
+            <min_angle>-0.2617993877991494</min_angle>
+            <max_angle>0.2617993877991494</max_angle>
           </vertical>
         </scan>
@@ -473,5 +473,5 @@
     <origin
       xyz="0 0.195 0.39805"
-      rpy="0 0 0" />
+      rpy="-1.57 0 0" />
     <parent
       link="chassis_link" />
@@ -577,5 +577,5 @@
   <joint
     name="arm_base_turret_joint"
-    type="revolute">
+    type="continuous">
     <origin
       xyz="-0.094203 0.07189 0.08635"
@@ -587,9 +587,4 @@
     <axis
       xyz="0 0 1" />
-    <limit
-      lower="-3.14"
-      upper="3.14"
-      effort="0"
-      velocity="0" />
     <dynamics
       damping="0.1"
@@ -638,5 +633,5 @@
   <joint
     name="arm_mid_joint"
-    type="revolute">
+    type="continuous">
     <origin
       xyz="0 0.6152 -0.020262"
@@ -648,9 +643,4 @@
     <axis
       xyz="0 0 -1" />
-    <limit
-      lower="-3.14"
-      upper="3.14"
-      effort="0"
-      velocity="0" />
     <dynamics
       damping="0.1"
@@ -699,5 +689,5 @@
   <joint
     name="arm_end_effector_turn_joint"
-    type="revolute">
+    type="continuous">
     <origin
       xyz="0.5747 -0.062022 0.05667"
@@ -709,9 +699,4 @@
     <axis
       xyz="0 0 -1" />
-    <limit
-      lower="-3.14"
-      upper="3.14"
-      effort="0"
-      velocity="0" />
     <dynamics
       damping="0.4"
@@ -833,4 +818,44 @@
       <state_interface name="position"></state_interface>
     </joint>
+    <joint name="arm_turret_joint">
+      <command_interface name = "position">
+        <param name="min">-3.14</param>
+        <param name="max">3.14</param>
+      </command_interface>
+      <state_interface name="position"></state_interface>
+      <state_interface name="velocity"></state_interface>
+    </joint>
+    <joint name="arm_base_turret_joint">
+      <command_interface name = "position">
+        <param name="min">-3.14</param>
+        <param name="max">3.14</param>
+      </command_interface>
+      <state_interface name="position"></state_interface>
+      <state_interface name="velocity"></state_interface>
+    </joint>
+    <joint name="arm_mid_joint">
+      <command_interface name = "position">
+        <param name="min">-10</param>
+        <param name="max">10</param>
+      </command_interface>
+      <state_interface name="position"></state_interface>
+      <state_interface name="velocity"></state_interface>
+    </joint>
+    <joint name="arm_end_effector_turn_joint">
+      <command_interface name = "position">
+        <param name="min">-10</param>
+        <param name="max">10</param>
+      </command_interface>
+      <state_interface name="position"></state_interface>
+      <state_interface name="velocity"></state_interface>
+    </joint>
+    <joint name="arm_end_effector_spin_joint">
+      <command_interface name = "position">
+        <param name="min">-10</param>
+        <param name="max">10</param>
+      </command_interface>
+      <state_interface name="position"></state_interface>
+      <state_interface name="velocity"></state_interface>
+    </joint>
   </ros2_control>
 </robot>

Commit message: update urdf

File: urdf/robot_description.urdf.xacro (robot description, xacro)
@@ -101,6 +101,6 @@
       xyz="0 0 -1" />
     <limit
-      lower="-1.57"
-      upper="1.57"
+      lower="-0.261799"
+      upper="0.261799"
       effort="0"
       velocity="0" />
@@ -274,6 +274,6 @@
       xyz="0 0 -1" />
     <limit
-      lower="-1.57"
-      upper="1.57"
+      lower="-0.261799"
+      upper="0.261799"
       effort="0"
       velocity="0" />
@@ -758,23 +758,4 @@
       damping="0.4" />
   </joint>
-  <!-- <gazebo> -->
-    <!-- <plugin filename="gz-sim-diff-drive-system" name="gz::sim::systems::DiffDrive"> -->
-      <!-- <left_joint>front_left_joint</left_joint> -->
-      <!-- <left_joint>rear_left_joint</left_joint> -->
-      <!-- <right_joint>front_right_joint</right_joint> -->
-      <!-- <right_joint>rear_right_joint</right_joint> -->
-      <!-- <wheel_separation>0.4</wheel_separation> -->
-      <!-- <wheel_radius>0.15</wheel_radius> -->
-      <!-- <publish_odom>true</publish_odom> -->
-      <!-- <publish_odom_tf>true</publish_odom_tf> -->
-      <!-- <publish_wheel_tf>true</publish_wheel_tf> -->
-      <!-- <odom_publish_frequency>50</odom_publish_frequency> -->
-      <!-- <topic>/cmd_vel</topic> -->
-      <!-- <odom_topic>/odom</odom_topic> -->
-      <!-- <tf_topic>/tf</tf_topic> -->
-      <!-- <frame_id>odom</frame_id> -->
-      <!-- <child_frame_id>base_link</child_frame_id> -->
-    <!-- </plugin> -->
-  <!-- </gazebo> -->
   <gazebo>
     <plugin filename="libgz_ros2_control-system.so" name="gz_ros2_control::GazeboSimROS2ControlPlugin">
@@ -786,4 +767,20 @@
       <plugin>gz_ros2_control/GazeboSimSystem</plugin>
     </hardware>
+    <joint name="left_rotatable_joint">
+      <command_interface name="position">
+        <param name="min">-0.261799</param>
+        <param name="max">0.261799</param>
+      </command_interface>
+      <state_interface name="position"/>
+      <state_interface name="velocity"/>
+    </joint>
+    <joint name="right_rotatable_joint">
+      <command_interface name="position">
+        <param name="min">-0.261799</param>
+        <param name="max">0.261799</param>
+      </command_interface>
+      <state_interface name="position"/>
+      <state_interface name="velocity"/>
+    </joint>
     <joint name="front_right_joint">
       <command_interface name="velocity">

Commit message: start to integrate moveit

File: urdf/robot_description.urdf.xacro (robot description, xacro)
@@ -277,5 +277,5 @@
       upper="0.261799"
       effort="0"
-      velocity="0" />
+      velocity="0.57" />
     <dynamics
       damping="0.4"
@@ -534,4 +534,5 @@
       damping="0.1"
       friction="0.1" />
+      <limit effort="100.0" lower="-3.14" upper="3.14" velocity="1.57"/>
   </joint>
   <link
@@ -590,4 +591,5 @@
       damping="0.1"
       friction="0.1" />
+      <limit effort="100.0" lower="-3.14" upper="3.14" velocity="1.57"/>
   </joint>
   <link
@@ -646,4 +648,5 @@
       damping="0.1"
       friction="0.1" />
+    <limit effort="100.0" lower="-1.57" upper="1.57" velocity="1.57"/>
   </joint>
   <link
@@ -702,4 +705,5 @@
       damping="0.4"
       friction="0.2" />
+      <limit effort="100.0" lower="-3.14" upper="3.14" velocity="1.57"/>
   </joint>
   <link
@@ -757,4 +761,5 @@
     <dynamics
       damping="0.4" />
+      <limit effort="100.0" lower="-3.14" upper="3.14" velocity="1.57"/>
   </joint>
   <gazebo>

Commit message: add gps

File: urdf/robot_description.urdf.xacro (robot description, xacro)
@@ -3,4 +3,11 @@
   name="tros_sldworks_pkg">
   <link name="base_link"></link>
+  <link name="gps_link">
+    <inertial>
+      <mass value="0.001"/>
+      <origin xyz="0 0 0" rpy="0 0 0"/>
+      <inertia ixx="0.0001" ixy="0" ixz="0" iyy="0.0001" iyz="0" izz="0.0001"/>
+    </inertial>
+  </link>
   <link
     name="chassis_link">
@@ -468,4 +475,29 @@
     </sensor>
   </gazebo>
+<gazebo reference="gps_link">
+  <sensor name="navsat" type="navsat">
+    <always_on>true</always_on>
+    <update_rate>1</update_rate>
+    <topic>gps/fix</topic>
+    <gz_frame_id>gps_link</gz_frame_id>
+    <plugin filename="gz-sim-navsat-system" name="gz::sim::systems::NavSat"/>
+    <navsat>
+      <position_sensing>
+        <horizontal>
+          <noise type="gaussian">
+            <mean>0.0</mean>
+            <stddev>0.0</stddev>
+          </noise>
+        </horizontal>
+        <vertical>
+          <noise type="gaussian">
+            <mean>0.0</mean>
+            <stddev>0.0</stddev>
+          </noise>
+        </vertical>
+      </position_sensing>
+    </navsat>
+  </sensor>
+</gazebo>
   <joint
     name="lidar_joint"
@@ -478,4 +510,9 @@
     <child
       link="lidar_link" />
+  </joint>
+  <joint name="gps_joint" type="fixed">
+    <parent link="base_link"/>
+    <child link="gps_link"/>
+    <origin xyz="-0.05 0 0.05" rpy="0 0 0"/>
   </joint>
   <link

Commit message: add camera and aruco

File: urdf/robot_description.urdf.xacro (robot description, xacro)
@@ -2,4 +2,5 @@
 <robot xmlns:xacro="http://ros.org"
   name="tros_sldworks_pkg">
+  <xacro:property name="rotatable_link_limit" value="0.0872665" />
   <link name="base_link"></link>
   <link name="gps_link">
@@ -55,4 +56,56 @@
     <origin xyz="0.0 0.0 0.0" rpy="1.5708 0 0"/>
   </joint>
+  <link name="camera_link">
+  <visual>
+    <geometry>
+      <box size="0.03 0.05 0.03"/>
+    </geometry>
+    <material name="black">
+      <color rgba="0.1 0.1 0.1 1"/>
+    </material>
+  </visual>
+  <collision>
+    <geometry>
+      <box size="0.03 0.05 0.03"/>
+    </geometry>
+  </collision>
+  <inertial>
+    <mass value="0.05"/>
+    <origin xyz="0 0 0" rpy="0 0 0"/>
+    <inertia ixx="0.00001" ixy="0" ixz="0" iyy="0.00001" iyz="0" izz="0.00001"/>
+  </inertial>
+</link>
+<joint name="camera_joint" type="fixed">
+  <parent link="chassis_link"/>
+  <child link="camera_link"/>
+  <origin xyz="0.0 0.025 -0.165" rpy="-1.57079632679 1.57079632679 0"/> <!-- Adjust position (x, y, z) relative to chassis -->
+</joint>
+<!-- Optical Link to align Gazebo frame (X-forward, Y-left, Z-up) with ROS Optical frame (X-right, Y-down, Z-forward) -->
+<link name="camera_optical_link"/>
+<joint name="camera_optical_joint" type="fixed">
+  <parent link="camera_link"/>
+  <child link="camera_optical_link"/>
+  <origin xyz="0 0 0" rpy="-1.57079632679 0 -1.57079632679"/> <!-- -pi/2 roll, -pi/2 yaw -->
+</joint>
+<gazebo reference="camera_link">
+  <sensor name="camera" type="camera">
+    <always_on>true</always_on>
+    <update_rate>30</update_rate>
+    <topic>chassis_camera/image_raw</topic>
+    <gz_frame_id>camera_optical_link</gz_frame_id>
+    <camera>
+      <horizontal_fov>1.21</horizontal_fov> <!-- ~70 degrees Field of View -->
+      <image>
+        <width>1600</width>
+        <height>1200</height>
+        <format>R8G8B8</format>
+      </image>
+      <clip>
+        <near>0.1</near>
+        <far>100.0</far>
+      </clip>
+    </camera>
+  </sensor>
+</gazebo>
   <link
     name="left_rotatable_link">
@@ -108,6 +161,6 @@
       xyz="0 0 -1" />
     <limit
-      lower="-0.261799"
-      upper="0.261799"
+      lower="-${rotatable_link_limit}"
+      upper="${rotatable_link_limit}"
       effort="0"
       velocity="0" />
@@ -281,6 +334,6 @@
       xyz="0 0 -1" />
     <limit
-      lower="-0.261799"
-      upper="0.261799"
+      lower="-${rotatable_link_limit}"
+      upper="${rotatable_link_limit}"
       effort="0"
       velocity="0.57" />
@@ -811,6 +864,6 @@
     <joint name="left_rotatable_joint">
       <command_interface name="position">
-        <param name="min">-0.261799</param>
-        <param name="max">0.261799</param>
+        <param name="min">-${rotatable_link_limit}</param>
+        <param name="max">${rotatable_link_limit}</param>
       </command_interface>
       <state_interface name="position"/>
@@ -819,6 +872,6 @@
     <joint name="right_rotatable_joint">
       <command_interface name="position">
-        <param name="min">-0.261799</param>
-        <param name="max">0.261799</param>
+        <param name="min">-${rotatable_link_limit}</param>
+        <param name="max">${rotatable_link_limit}</param>
       </command_interface>
       <state_interface name="position"/>

Commit message: add dual ekf, needs tuning

File: urdf/robot_description.urdf.xacro (robot description, xacro)
@@ -11,4 +11,24 @@
     </inertial>
   </link>
+  <link name="imu_link">
+  <visual>
+    <geometry>
+      <box size="0.02 0.02 0.005"/> <!-- Small board dimensions -->
+    </geometry>
+    <material name="blue">
+      <color rgba="0.0 0.0 0.8 1.0"/>
+    </material>
+  </visual>
+  <collision>
+    <geometry>
+      <box size="0.02 0.02 0.005"/>
+    </geometry>
+  </collision>
+  <inertial>
+    <mass value="0.005"/>
+    <origin xyz="0 0 0" rpy="0 0 0"/>
+    <inertia ixx="0.000001" ixy="0" ixz="0" iyy="0.000001" iyz="0" izz="0.000001"/>
+  </inertial>
+</link>
   <link
     name="chassis_link">
@@ -51,9 +71,10 @@
     </collision>
   </link>
-  <joint name="chassis_joint" type="fixed">
-    <parent link="base_link"/>
-    <child link="chassis_link"/>
-    <origin xyz="0.0 0.0 0.0" rpy="1.5708 0 0"/>
-  </joint>
+<joint name="chassis_joint" type="fixed">
+  <parent link="base_link"/>
+  <child link="chassis_link"/>
+  <!-- Added -1.5708 to the Yaw (last value) -->
+  <origin xyz="0.0 0.0 0.0" rpy="1.5708 0 -1.5708"/>
+</joint>
   <link name="camera_link">
   <visual>
@@ -88,4 +109,9 @@
   <origin xyz="0 0 0" rpy="-1.57079632679 0 -1.57079632679"/> <!-- -pi/2 roll, -pi/2 yaw -->
 </joint>
+<joint name="imu_joint" type="fixed">
+  <parent link="chassis_link"/>
+  <child link="imu_link"/>
+  <origin xyz="0.0 0.0 0.05" rpy="0 0 0"/> <!-- Adjust position (x, y, z) relative to chassis -->
+</joint>
 <gazebo reference="camera_link">
   <sensor name="camera" type="camera">
@@ -106,4 +132,56 @@
       </clip>
     </camera>
+  </sensor>
+</gazebo>
+<gazebo reference="imu_link">
+  <sensor name="bno055_imu" type="imu">
+    <always_on>true</always_on>
+    <update_rate>100</update_rate> <!-- BNO055 runs natively at 100 Hz -->
+    <topic>imu/data</topic>
+    <gz_frame_id>imu_link</gz_frame_id>
+    <!-- Required Gazebo IMU System Plugin -->
+    <plugin filename="gz-sim-imu-system" name="gz::sim::systems::Imu"/>
+    <imu>
+      <angular_velocity>
+        <x>
+          <noise type="gaussian">
+            <mean>0.0</mean>
+            <stddev>0.0002</stddev> <!-- ~0.01 deg/s noise -->
+          </noise>
+        </x>
+        <y>
+          <noise type="gaussian">
+            <mean>0.0</mean>
+            <stddev>0.0002</stddev>
+          </noise>
+        </y>
+        <z>
+          <noise type="gaussian">
+            <mean>0.0</mean>
+            <stddev>0.0002</stddev>
+          </noise>
+        </z>
+      </angular_velocity>
+      <linear_acceleration>
+        <x>
+          <noise type="gaussian">
+            <mean>0.0</mean>
+            <stddev>0.01</stddev> <!-- ~1 mg noise -->
+          </noise>
+        </x>
+        <y>
+          <noise type="gaussian">
+            <mean>0.0</mean>
+            <stddev>0.01</stddev>
+          </noise>
+        </y>
+        <z>
+          <noise type="gaussian">
+            <mean>0.0</mean>
+            <stddev>0.01</stddev>
+          </noise>
+        </z>
+      </linear_acceleration>
+    </imu>
   </sensor>
 </gazebo>
@@ -531,5 +609,5 @@
   <sensor name="navsat" type="navsat">
     <always_on>true</always_on>
-    <update_rate>1</update_rate>
+    <update_rate>10</update_rate>
     <topic>gps/fix</topic>
     <gz_frame_id>gps_link</gz_frame_id>
